File: hardware/final_outline.kicad_pcb (KiCad board)
At the start: 2 copper layers, 99.5 x 75 mm, 44 parts, among them P001 CANCONNECTOR, P002 CONN_01X14, P100 ISP, P101 DEBUG_LED, Q601 2N7002, Q602 2N7002, U401 MCP2551-I/SN, U402 MCP2515_TSSOP, U403 LPC11C14, U404 MCP2551-I/SN, U501 MCP1755-33, U502 MCP1755-5, U601 MAX232

Commit message: Final version of board
Parts:
- removed Q601, Q602: 2N7002, TO_SOT_Packages_SMD:SOT-23
- added ?: , OSHW-logo:OSHW-logo_silkscreen-front_10mm, F.Cu at (196.2, 119.6)
- added ?: , MITEVT_AUTOMOTIVECON:EVT-LOGO, F.Cu at (196.2, 107.8)
- added U602: SN74HCT125, Housings_SOIC:SOIC-14_3.9x8.7mm_Pitch1.27mm, F.Cu at (158.6, 85.4)
- R601: value 20k -> 20K
- moved C407 5.75 mm to (164.5, 100.5), turned to 270 degrees
- moved R601 1.40 mm to (161.4, 78.2)
- moved C408 1.02 mm to (167.5, 100.5), turned to 270 degrees
- moved C601 0.18 mm to (176.0, 84.0)
Connections:
- R601 pad 1: Net-(Q601-Pad2) -> +5V
- R601 pad 2: GND -> Net-(R601-Pad2)
- U601 pad 11: Net-(Q601-Pad2) -> Net-(R601-Pad2)
Routing:
- net +5V: track 201.0 -> 181.0 mm, vias 4 -> 2
- net Net-(Q601-Pad2): track 19.5 -> 0.00 mm
- net Net-(R601-Pad2): track 0.00 -> 15.4 mm
- net GND: track 49.4 -> 57.9 mm, vias 11 -> 15
- net +3V3: track 92.7 -> 85.1 mm
- net /BACK_PANEL/RS232_MSG: track 36.9 -> 42.1 mm
- net /Micro_Controller/RS232_CTRL: track 49.3 -> 45.4 mm
- net /FRONT_PANEL/TXD: track 73.5 -> 76.3 mm
- net +12V: track 29.9 -> 28.7 mm
- net (no net): track 2.50 -> 3.53 mm, vias 1 -> 0
Other:
- board text added: "Motor Interface - June 16, 2016"
